File: KiCad/Car_bs_controller_nex_mega/Digital_inputs.sch (KiCad schematic (older format))
At the start: 42 parts

Commit message: big update
Parts:
- removed D11, D12, D13, D14, D15, D16: SMAJ18, Diode_SMD:D_SMA, symbol Device:D_TVS
- removed R16, R17, R18, R19, R20, R21: 100R, Resistor_SMD:R_0805_2012Metric, symbol Device:R
- added D22, D23, D24, D25, D26, D27: BAV99, Package_TO_SOT_SMD:SOT-23, symbol Diode:BAV99
- C14: renamed from C20; footprint Capacitor_SMD:C_0805_2012Metric -> Capacitor_SMD:C_0603_1608Metric_Pad1.08x0.95mm_HandSolder; symbol Device:C -> Car_bs_controller_nex_mega-rescue:C-Device
- C15: renamed from C21; footprint Capacitor_SMD:C_0805_2012Metric -> Capacitor_SMD:C_0603_1608Metric_Pad1.08x0.95mm_HandSolder; symbol Device:C -> Car_bs_controller_nex_mega-rescue:C-Device
- C16: renamed from C22; footprint Capacitor_SMD:C_0805_2012Metric -> Capacitor_SMD:C_0603_1608Metric_Pad1.08x0.95mm_HandSolder; symbol Device:C -> Car_bs_controller_nex_mega-rescue:C-Device
- C17: renamed from C23; footprint Capacitor_SMD:C_0805_2012Metric -> Capacitor_SMD:C_0603_1608Metric_Pad1.08x0.95mm_HandSolder; symbol Device:C -> Car_bs_controller_nex_mega-rescue:C-Device
- C18: renamed from C24; footprint Capacitor_SMD:C_0805_2012Metric -> Capacitor_SMD:C_0603_1608Metric_Pad1.08x0.95mm_HandSolder; symbol Device:C -> Car_bs_controller_nex_mega-rescue:C-Device
- C19: renamed from C25; footprint Capacitor_SMD:C_0805_2012Metric -> Capacitor_SMD:C_0603_1608Metric_Pad1.08x0.95mm_HandSolder; symbol Device:C -> Car_bs_controller_nex_mega-rescue:C-Device
- D10: renamed from D17; symbol Diode:LL4148 -> Car_bs_controller_nex_mega-rescue:LL4148-Diode
- D11: renamed from D18; symbol Diode:LL4148 -> Car_bs_controller_nex_mega-rescue:LL4148-Diode
- D12: renamed from D19; symbol Diode:LL4148 -> Car_bs_controller_nex_mega-rescue:LL4148-Diode
- D13: renamed from D20; symbol Diode:LL4148 -> Car_bs_controller_nex_mega-rescue:LL4148-Diode
- D14: renamed from D21; symbol Diode:LL4148 -> Car_bs_controller_nex_mega-rescue:LL4148-Diode
- D15: renamed from D22; symbol Diode:LL4148 -> Car_bs_controller_nex_mega-rescue:LL4148-Diode
- D16: renamed from D23; symbol Device:D_Zener -> Car_bs_controller_nex_mega-rescue:D_Zener-Device
- D17: renamed from D24; symbol Device:D_Zener -> Car_bs_controller_nex_mega-rescue:D_Zener-Device
- D18: renamed from D25; symbol Device:D_Zener -> Car_bs_controller_nex_mega-rescue:D_Zener-Device
- D19: renamed from D26; symbol Device:D_Zener -> Car_bs_controller_nex_mega-rescue:D_Zener-Device
- D20: renamed from D27; symbol Device:D_Zener -> Car_bs_controller_nex_mega-rescue:D_Zener-Device
- D21: renamed from D28; symbol Device:D_Zener -> Car_bs_controller_nex_mega-rescue:D_Zener-Device
- R10: renamed from R26; footprint Resistor_SMD:R_0805_2012Metric -> Resistor_SMD:R_0603_1608Metric_Pad0.98x0.95mm_HandSolder; symbol Device:R -> Car_bs_controller_nex_mega-rescue:R-Device
- R11: renamed from R27; footprint Resistor_SMD:R_0805_2012Metric -> Resistor_SMD:R_0603_1608Metric_Pad0.98x0.95mm_HandSolder; symbol Device:R -> Car_bs_controller_nex_mega-rescue:R-Device
- R12: renamed from R28; footprint Resistor_SMD:R_0805_2012Metric -> Resistor_SMD:R_0603_1608Metric_Pad0.98x0.95mm_HandSolder; symbol Device:R -> Car_bs_controller_nex_mega-rescue:R-Device
- R13: renamed from R29; footprint Resistor_SMD:R_0805_2012Metric -> Resistor_SMD:R_0603_1608Metric_Pad0.98x0.95mm_HandSolder; symbol Device:R -> Car_bs_controller_nex_mega-rescue:R-Device
- R14: renamed from R30; footprint Resistor_SMD:R_0805_2012Metric -> Resistor_SMD:R_0603_1608Metric_Pad0.98x0.95mm_HandSolder; symbol Device:R -> Car_bs_controller_nex_mega-rescue:R-Device
- R15: renamed from R31; footprint Resistor_SMD:R_0805_2012Metric -> Resistor_SMD:R_0603_1608Metric_Pad0.98x0.95mm_HandSolder; symbol Device:R -> Car_bs_controller_nex_mega-rescue:R-Device
- R16: renamed from R32; footprint Resistor_SMD:R_0805_2012Metric -> Resistor_SMD:R_0603_1608Metric_Pad0.98x0.95mm_HandSolder; symbol Device:R -> Car_bs_controller_nex_mega-rescue:R-Device
- R17: renamed from R33; footprint Resistor_SMD:R_0805_2012Metric -> Resistor_SMD:R_0603_1608Metric_Pad0.98x0.95mm_HandSolder; symbol Device:R -> Car_bs_controller_nex_mega-rescue:R-Device
- R6: renamed from R22; footprint Resistor_SMD:R_0805_2012Metric -> Resistor_SMD:R_0603_1608Metric_Pad0.98x0.95mm_HandSolder; symbol Device:R -> Car_bs_controller_nex_mega-rescue:R-Device
- R7: renamed from R23; value 22k -> 15k; footprint Resistor_SMD:R_0805_2012Metric -> Resistor_SMD:R_0603_1608Metric_Pad0.98x0.95mm_HandSolder; symbol Device:R -> Car_bs_controller_nex_mega-rescue:R-Device
- R8: renamed from R24; footprint Resistor_SMD:R_0805_2012Metric -> Resistor_SMD:R_0603_1608Metric_Pad0.98x0.95mm_HandSolder; symbol Device:R -> Car_bs_controller_nex_mega-rescue:R-Device
- R9: renamed from R25; value 22k -> 15k; footprint Resistor_SMD:R_0805_2012Metric -> Resistor_SMD:R_0603_1608Metric_Pad0.98x0.95mm_HandSolder; symbol Device:R -> Car_bs_controller_nex_mega-rescue:R-Device
Connections:
- net DOOR_SWITCH_INPUT: now also D13.1 (K)
- net GND: now also D22.1 (K), D23.1 (K), D24.1 (K), D25.1 (K), D26.1 (K), D27.1 (K)
- net IGNITION_SWITCH_INPUT: now also D12.2 (A)
- net LOW_WASHER_WATER_LEVEL_INPUT: now also D15.1 (K)
- net MCU_door_switch_input: now also D24.3 (K)
- net MCU_ignition_switch_input: now also D26.3 (K)
- net MCU_low_washer_water_level_input: now also D27.3 (K)
- net MCU_proximity_input: now also D25.3 (K)
- net MCU_spare_input_1: now also D22.3 (K)
- net MCU_water_flow_sensor: now also D23.3 (K)
- net PROXIMITY_SENSOR_INPUT: now also D14.1 (K)
- net SPARE_INPUT_1: now also D11.2 (A)
- net WATER_FLOW_SENSOR_INPUT: now also D10.1 (K)
- new net +5v_FROM_MCU: D22.2 (A), D23.2 (A), D24.2 (A), D25.2 (A), D26.2 (A), D27.2 (A)
