File: KiCad/Car_bs_controller_nex_mega/Links.sch (KiCad schematic (older format))
At the start: 46 parts, among them Q1 BSS138, SW1 SW_Push, U4 ADM705, U5 MAX485E

Commit message: Update
Parts:
- LS1: symbol PKLCS1212E4001-R1:PKLCS1212E4001-R1 -> Car_bs_controller_nex_mega-rescue:PKLCS1212E4001-R1-PKLCS1212E4001-R1
- U4: symbol ADM705:ADM705 -> Car_bs_controller_nex_mega-rescue:ADM705-ADM705
Changed lines of the file:
@@
 Connection ~ 9000 3900
 $Comp
-L PKLCS1212E4001-R1:PKLCS1212E4001-R1 LS1
+L Car_bs_controller_nex_mega-rescue:PKLCS1212E4001-R1-PKLCS1212E4001-R1 LS1
 U 1 1 60150DF8
 P 9850 3550
@@
 	9600 3350 9600 3450
 $Comp
-L ADM705:ADM705 U?
+L Car_bs_controller_nex_mega-rescue:ADM705-ADM705 U?
 U 1 1 6017DAE3
 P 3950 5550

Commit message: big update
Parts:
- removed C27: 1mk, Resistor_SMD:R_0805_2012Metric, symbol Device:C
- removed R42, R43: 22R, Resistor_SMD:R_0805_2012Metric, symbol Device:R
- removed R60: 120R, Resistor_SMD:R_1206_3216Metric, symbol Device:R
- added C21: 10mk, Capacitor_Tantalum_SMD:CP_EIA-7343-15_Kemet-W_Pad2.25x2.55mm_HandSolder, symbol Car_bs_controller_nex_mega-rescue:C-Device
- added C23: 1n, Resistor_SMD:R_0603_1608Metric_Pad0.98x0.95mm_HandSolder, symbol Car_bs_controller_nex_mega-rescue:C-Device
- added JP1: SolderJumper_2_Open, Jumper:SolderJumper-2_P1.3mm_Open_RoundedPad1.0x1.5mm, symbol Jumper:SolderJumper_2_Open
- added L2, L3: BLN, Inductor_SMD:L_0805_2012Metric_Pad1.15x1.40mm_HandSolder, symbol Device:L
- added R27: 1k, Resistor_SMD:R_0603_1608Metric_Pad0.98x0.95mm_HandSolder, symbol Car_bs_controller_nex_mega-rescue:R-Device
- added R28: 220R, Resistor_SMD:R_0603_1608Metric_Pad0.98x0.95mm_HandSolder, symbol Car_bs_controller_nex_mega-rescue:R-Device
- added R38: 470R, Resistor_SMD:R_0603_1608Metric_Pad0.98x0.95mm_HandSolder, symbol Car_bs_controller_nex_mega-rescue:R-Device
- added R45: 1k, Resistor_SMD:R_0805_2012Metric_Pad1.20x1.40mm_HandSolder, symbol Car_bs_controller_nex_mega-rescue:R-Device
- C22: renamed from C26; symbol Device:C -> Car_bs_controller_nex_mega-rescue:C-Device
- C24: renamed from C28; value 4m7 -> 10m; footprint Capacitor_SMD:C_1206_3216Metric -> Capacitor_SMD:C_1210_3225Metric_Pad1.33x2.70mm_HandSolder; symbol Device:C -> Car_bs_controller_nex_mega-rescue:C-Device
- C25: renamed from C29; footprint Capacitor_SMD:C_0805_2012Metric -> Capacitor_SMD:C_0603_1608Metric_Pad1.08x0.95mm_HandSolder; symbol Device:C -> Car_bs_controller_nex_mega-rescue:C-Device
- D28: renamed from D29; symbol Diode:BAV99 -> Car_bs_controller_nex_mega-rescue:BAV99-Diode
- D29: renamed from D30; symbol Diode:BAV99 -> Car_bs_controller_nex_mega-rescue:BAV99-Diode
- D30: renamed from D32; symbol Device:LED -> Car_bs_controller_nex_mega-rescue:LED-Device
- D31: symbol Device:LED -> Car_bs_controller_nex_mega-rescue:LED-Device
- D32: renamed from D33; symbol Device:LED -> Car_bs_controller_nex_mega-rescue:LED-Device
- D33: renamed from D34; symbol Device:LED -> Car_bs_controller_nex_mega-rescue:LED-Device
- D34: renamed from D35; symbol Device:LED -> Car_bs_controller_nex_mega-rescue:LED-Device
- D35: renamed from D36; symbol Device:D_TVS -> Car_bs_controller_nex_mega-rescue:D_TVS-Device
- D36: renamed from D37; symbol Device:D_TVS -> Car_bs_controller_nex_mega-rescue:D_TVS-Device
- Q1: symbol Transistor_FET:BSS138 -> Car_bs_controller_nex_mega-rescue:BSS138-Transistor_FET
- R18: renamed from R34; symbol Device:R -> Car_bs_controller_nex_mega-rescue:R-Device
- R19: renamed from R35; symbol Device:R -> Car_bs_controller_nex_mega-rescue:R-Device
- R20: renamed from R36; symbol Device:R -> Car_bs_controller_nex_mega-rescue:R-Device
- R21: renamed from R37; footprint Resistor_SMD:R_0603_1608Metric -> Resistor_SMD:R_0603_1608Metric_Pad0.98x0.95mm_HandSolder; symbol Device:R -> Car_bs_controller_nex_mega-rescue:R-Device
- R22: renamed from R40; footprint Resistor_SMD:R_0603_1608Metric -> Resistor_SMD:R_0603_1608Metric_Pad0.98x0.95mm_HandSolder; symbol Device:R -> Car_bs_controller_nex_mega-rescue:R-Device
- R23: renamed from R38; footprint Resistor_SMD:R_0805_2012Metric -> Resistor_SMD:R_0603_1608Metric_Pad0.98x0.95mm_HandSolder; symbol Device:R -> Car_bs_controller_nex_mega-rescue:R-Device
- R24: renamed from R41; symbol Device:R -> Car_bs_controller_nex_mega-rescue:R-Device
- R25: renamed from R39; symbol Device:R -> Car_bs_controller_nex_mega-rescue:R-Device
- R26: renamed from R44; footprint Resistor_SMD:R_0603_1608Metric -> Resistor_SMD:R_0603_1608Metric_Pad0.98x0.95mm_HandSolder; symbol Device:R -> Car_bs_controller_nex_mega-rescue:R-Device
- R29: renamed from R45; footprint Resistor_SMD:R_0603_1608Metric -> Resistor_SMD:R_0603_1608Metric_Pad0.98x0.95mm_HandSolder; symbol Device:R -> Car_bs_controller_nex_mega-rescue:R-Device
- R30: renamed from R46; footprint Resistor_SMD:R_0603_1608Metric -> Resistor_SMD:R_0603_1608Metric_Pad0.98x0.95mm_HandSolder; symbol Device:R -> Car_bs_controller_nex_mega-rescue:R-Device
- R31: renamed from R48; footprint Resistor_SMD:R_0805_2012Metric -> Resistor_SMD:R_0603_1608Metric_Pad0.98x0.95mm_HandSolder; symbol Device:R -> Car_bs_controller_nex_mega-rescue:R-Device
- R32: renamed from R47; value 2k2 -> 1k2; symbol Device:R -> Car_bs_controller_nex_mega-rescue:R-Device
- R33: renamed from R49; footprint Resistor_SMD:R_0805_2012Metric -> Resistor_SMD:R_0603_1608Metric_Pad0.98x0.95mm_HandSolder; symbol Device:R -> Car_bs_controller_nex_mega-rescue:R-Device
- R34: renamed from R50; value 2k2 -> 1k; symbol Device:R -> Car_bs_controller_nex_mega-rescue:R-Device
- R35: renamed from R51; footprint Resistor_SMD:R_0805_2012Metric -> Resistor_SMD:R_0603_1608Metric_Pad0.98x0.95mm_HandSolder; symbol Device:R -> Car_bs_controller_nex_mega-rescue:R-Device
- R36: renamed from R52; value 2k2 -> 1k; symbol Device:R -> Car_bs_controller_nex_mega-rescue:R-Device
- R37: renamed from R53; footprint Resistor_SMD:R_0603_1608Metric -> Resistor_SMD:R_0603_1608Metric_Pad0.98x0.95mm_HandSolder; symbol Device:R -> Car_bs_controller_nex_mega-rescue:R-Device
- R39: renamed from R54; footprint Resistor_SMD:R_0805_2012Metric -> Resistor_SMD:R_0603_1608Metric_Pad0.98x0.95mm_HandSolder; symbol Device:R -> Car_bs_controller_nex_mega-rescue:R-Device
- R40: renamed from R55; footprint Resistor_SMD:R_0603_1608Metric -> Resistor_SMD:R_0603_1608Metric_Pad0.98x0.95mm_HandSolder; symbol Device:R -> Car_bs_controller_nex_mega-rescue:R-Device
- R41: renamed from R56; symbol Device:R -> Car_bs_controller_nex_mega-rescue:R-Device
- R42: renamed from R57; footprint Resistor_SMD:R_0805_2012Metric -> Resistor_SMD:R_0603_1608Metric_Pad0.98x0.95mm_HandSolder; symbol Device:R -> Car_bs_controller_nex_mega-rescue:R-Device
- R43: renamed from R58; symbol Device:R -> Car_bs_controller_nex_mega-rescue:R-Device
- R44: renamed from R59; symbol Device:R -> Car_bs_controller_nex_mega-rescue:R-Device
- RV1: symbol Device:R_POT -> Car_bs_controller_nex_mega-rescue:R_POT-Device
- SW1: symbol Switch:SW_Push -> Car_bs_controller_nex_mega-rescue:SW_Push-Switch
- U3: renamed from U5; symbol Interface_UART:MAX485E -> Car_bs_controller_nex_mega-rescue:MAX485E-Interface_UART
- renumbered U4 to U2
Connections:
- net 5V_sensors_stab is gone; now on net +5v_FROM_MCU: C24.1, C25.1, D33.2 (A), D34.2 (A), R31.1, R33.1, R35.1, R42.1, U3.8 (VCC)
- net +5v_FROM_MCU: now also C21.1
- net GND: now also C21.2, C23.2
- net MCU_button_on_board: now also R38.2; no longer SW1.1
- net MCU_one_wire_PIN: now also D28.3 (K), R23.2, R24.2, L2.2
- net MCU_pjon_bus_PIN: now also D29.3 (K), R25.1, L3.2
- net MCU_rst: now also JP1.2 (B); no longer U2.7 (RST)
- net at R21.1, RV1.1, RV1.2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: now also C23.1, R27.2
- net at R30.2, U2.5 (PFO): now also R27.1
- net at LS1.P, R41.1: now also R45.1
- net at LS1.N, Q1.3 (D): now also R45.2
- new net: L3.1, R20.1
- new net: L2.1, R19.1
- new net: R28.2, U2.7 (RST)
- new net: R38.1, SW1.1
- new net: JP1.1 (A), R28.1
Other:
- moved on the sheet: D28, D29, D30, D31, D32, LS1, R18, R19, R20, R23, R24, R25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
