File: KiCad/Car_bs_controller_nex_mega/Plugs.sch (KiCad schematic (older format))
At the start: 34 parts, among them J1 Power, J10 Encoder, J11 LCD_Nextion, J12 PUMP_RELAY, J13 LIGHT_RELAY, J14 LIGHT_RELAY, J15 I2C, J2 Inputs, J3 Proxy, J4 PJON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

Commit message: Update
Parts:
- J14: value LIGHT_RELAY -> CONVERTER_RELAY
Changed lines of the file:
@@
 P 9950 2350
 F 0 "J14" H 10030 2342 50  0000 L CNN
-F 1 "LIGHT_RELAY" H 10030 2251 50  0000 L CNN
+F 1 "CONVERTER_RELAY" H 10030 2251 50  0000 L CNN
 F 2 "Connector_Phoenix_MSTB:PhoenixContact_MSTBA_2,5_2-G_1x02_P5.00mm_Horizontal" H 9950 2350 50  0001 C CNN
 F 3 "~" H 9950 2350 50  0001 C CNN

Commit message: big update
Parts:
- removed F2: 200mA 5v, Fuse:Fuse_1210_3225Metric, symbol Device:Fuse
- removed F3, F4: 200mA, Fuse:Fuse_1210_3225Metric, symbol Device:Fuse
- added F4: 200mA 5v, Fuse:Fuse_1206_3216Metric_Pad1.42x1.75mm_HandSolder, symbol Car_bs_controller_nex_mega-rescue:Fuse-Device
- C26: renamed from C30; symbol Device:C -> Car_bs_controller_nex_mega-rescue:C-Device
- C27: renamed from C31; symbol Device:C -> Car_bs_controller_nex_mega-rescue:C-Device
- C28: renamed from C32; symbol Device:C -> Car_bs_controller_nex_mega-rescue:C-Device
- D41: renamed from D42; symbol Simulation_SPICE:DIODE -> Car_bs_controller_nex_mega-rescue:DIODE-Simulation_SPICE
- D42: renamed from D43; symbol Simulation_SPICE:DIODE -> Car_bs_controller_nex_mega-rescue:DIODE-Simulation_SPICE
- D43: renamed from D44; symbol Simulation_SPICE:DIODE -> Car_bs_controller_nex_mega-rescue:DIODE-Simulation_SPICE
- F2: renamed from F5; footprint Fuse:Fuse_1210_3225Metric -> Fuse:Fuse_1206_3216Metric_Pad1.42x1.75mm_HandSolder; symbol Device:Fuse -> Car_bs_controller_nex_mega-rescue:Fuse-Device
- F3: renamed from F6; footprint Fuse:Fuse_1210_3225Metric -> Fuse:Fuse_1206_3216Metric_Pad1.42x1.75mm_HandSolder; symbol Device:Fuse -> Car_bs_controller_nex_mega-rescue:Fuse-Device
- J1, J3, J4, J7: symbol Connector_Generic:Conn_01x03 -> Car_bs_controller_nex_mega-rescue:Conn_01x03-Connector_Generic
- J10, J2, J8: symbol Connector_Generic:Conn_01x05 -> Car_bs_controller_nex_mega-rescue:Conn_01x05-Connector_Generic
- J11: symbol Connector_Generic:Conn_01x04 -> Car_bs_controller_nex_mega-rescue:Conn_01x04-Connector_Generic
- J12: renamed from J15; symbol Connector_Generic:Conn_01x04 -> Car_bs_controller_nex_mega-rescue:Conn_01x04-Connector_Generic
- J13: renamed from J12; symbol Connector_Generic:Conn_01x02 -> Car_bs_controller_nex_mega-rescue:Conn_01x02-Connector_Generic
- J14: renamed from J13; symbol Connector_Generic:Conn_01x02 -> Car_bs_controller_nex_mega-rescue:Conn_01x02-Connector_Generic
- J15: renamed from J14; symbol Connector_Generic:Conn_01x02 -> Car_bs_controller_nex_mega-rescue:Conn_01x02-Connector_Generic
- J5, J6: symbol Connector_Generic:Conn_01x02 -> Car_bs_controller_nex_mega-rescue:Conn_01x02-Connector_Generic
- J9: symbol Connector_Generic:Conn_01x08 -> Car_bs_controller_nex_mega-rescue:Conn_01x08-Connector_Generic
- JP2: renamed from JP1; symbol Jumper:SolderJumper_3_Open -> Car_bs_controller_nex_mega-rescue:SolderJumper_3_Open-Jumper
- Q2: symbol Transistor_BJT:BC857 -> Car_bs_controller_nex_mega-rescue:BC857-Transistor_BJT
- R49: renamed from R64; footprint Resistor_SMD:R_0805_2012Metric -> Resistor_SMD:R_0603_1608Metric_Pad0.98x0.95mm_HandSolder; symbol Device:R -> Car_bs_controller_nex_mega-rescue:R-Device
- R50: renamed from R65; footprint Resistor_SMD:R_0603_1608Metric -> Resistor_SMD:R_0603_1608Metric_Pad0.98x0.95mm_HandSolder; symbol Device:R -> Car_bs_controller_nex_mega-rescue:R-Device
- R51: renamed from R66; symbol Device:R -> Car_bs_controller_nex_mega-rescue:R-Device
- R52: renamed from R77; symbol Device:R -> Car_bs_controller_nex_mega-rescue:R-Device
- R53: renamed from R78; symbol Device:R -> Car_bs_controller_nex_mega-rescue:R-Device
- RV5: symbol Device:R_POT -> Car_bs_controller_nex_mega-rescue:R_POT-Device
Connections:
- net +5v_FROM_MCU: now also F4.2; no longer J12.1 (Pin_1), R52.2, R53.2
- net CONVERTER_RELAY_COM: now also J15.2 (Pin_2); no longer J15.1 (Pin_1)
- net CONVERTER_RELAY_NO: now also J15.1 (Pin_1); no longer J15.2 (Pin_2)
- net LIGHT_RELAY_COM: now also J14.2 (Pin_2); no longer J14.1 (Pin_1)
- net LIGHT_RELAY_NO: now also J14.1 (Pin_1); no longer J14.2 (Pin_2)
- net PUMP_RELAY_COM: now also J13.2 (Pin_2); no longer J13.1 (Pin_1)
- net PUMP_RELAY_NO: now also J13.1 (Pin_1); no longer J13.2 (Pin_2)
- net at J3.1 (Pin_1): now also D42.2 (K)
- net at J4.1 (Pin_1): now also D41.2 (K)
- net at J7.1 (Pin_1): now also D43.2 (K)
- new net: F4.1, J12.1 (Pin_1), R52.2, R53.2
