File: KiCad/Car_bs_controller_nex_mega/Analog_input.sch (KiCad schematic (older format))
At the start: 19 parts, among them U7 TL431DBZ

Commit message: big update
Parts:
- removed D46, D48, D50: 2v4, Diode_SMD:D_MELF, symbol Device:D_Zener
- removed R70, R73, R76: 2k2, Resistor_SMD:R_0805_2012Metric, symbol Device:R
- added C30, C32, C35: 10n, Resistor_SMD:R_0603_1608Metric, symbol Car_bs_controller_nex_mega-rescue:C-Device
- added C33: 100n, Resistor_SMD:R_0603_1608Metric, symbol Car_bs_controller_nex_mega-rescue:C-Device
- added C34: 10mk, Capacitor_Tantalum_SMD:CP_EIA-6032-15_Kemet-U, symbol Device:CP
- added R59, R63, R67: 6k8, Resistor_SMD:R_0603_1608Metric_Pad0.98x0.95mm_HandSolder, symbol Car_bs_controller_nex_mega-rescue:R-Device
- added R60: 2k2, Resistor_SMD:R_0603_1608Metric_Pad0.98x0.95mm_HandSolder, symbol Car_bs_controller_nex_mega-rescue:R-Device
- added R61, R62, R64, R68: 10k, Resistor_SMD:R_0603_1608Metric_Pad0.98x0.95mm_HandSolder, symbol Car_bs_controller_nex_mega-rescue:R-Device
- added U6: MCP6004, Package_SO:SOIC-14_3.9x8.7mm_P1.27mm, symbol Amplifier_Operational:MCP6004
- C29: renamed from C33; symbol Device:C -> Car_bs_controller_nex_mega-rescue:C-Device
- C31: renamed from C34; symbol Device:C -> Car_bs_controller_nex_mega-rescue:C-Device
- D44: renamed from D45; symbol Diode:BAV99 -> Car_bs_controller_nex_mega-rescue:BAV99-Diode
- D45: renamed from D47; symbol Diode:BAV99 -> Car_bs_controller_nex_mega-rescue:BAV99-Diode
- D46: renamed from D49; symbol Diode:BAV99 -> Car_bs_controller_nex_mega-rescue:BAV99-Diode
- R54: renamed from R67; value 10k -> 39k; footprint Resistor_SMD:R_0805_2012Metric -> Resistor_SMD:R_0603_1608Metric_Pad0.98x0.95mm_HandSolder; symbol Device:R -> Car_bs_controller_nex_mega-rescue:R-Device
- R55: renamed from R68; value 1k -> 10k; footprint Resistor_SMD:R_0805_2012Metric -> Resistor_SMD:R_0603_1608Metric_Pad0.98x0.95mm_HandSolder; symbol Device:R -> Car_bs_controller_nex_mega-rescue:R-Device
- R56: renamed from R72; value 2k2 -> 1k; symbol Device:R -> Car_bs_controller_nex_mega-rescue:R-Device
- R57: renamed from R71; value 100R -> 10k; footprint Resistor_SMD:R_0805_2012Metric -> Resistor_SMD:R_0603_1608Metric_Pad0.98x0.95mm_HandSolder; symbol Device:R -> Car_bs_controller_nex_mega-rescue:R-Device
- R58: renamed from R69; value 150R -> 330R; symbol Device:R -> Car_bs_controller_nex_mega-rescue:R-Device
- R65: renamed from R74; value 10k -> 22k; footprint Resistor_SMD:R_0805_2012Metric -> Resistor_SMD:R_0603_1608Metric_Pad0.98x0.95mm_HandSolder; symbol Device:R -> Car_bs_controller_nex_mega-rescue:R-Device
- R66: renamed from R75; value 1k -> 10k; footprint Resistor_SMD:R_0805_2012Metric -> Resistor_SMD:R_0603_1608Metric_Pad0.98x0.95mm_HandSolder; symbol Device:R -> Car_bs_controller_nex_mega-rescue:R-Device
- U5: renamed from U7; symbol Reference_Voltage:TL431DBZ -> Car_bs_controller_nex_mega-rescue:TL431DBZ-Reference_Voltage
Connections:
- net +5v_FROM_MCU: now also D44.2 (A), D45.2 (A), D46.2 (A), C33.1, C34.1, U6.4 (V+)
- net GND: now also C30.2, C32.2, C33.2, C34.2, C35.2, R60.1, R61.1, R64.1, R68.1, U6.11 (V-)
- net MCU_resistive_sensor_0_190: now also R63.1, R64.2; no longer D45.3 (K), R57.1
- net MCU_sensors_voltage_test_input: now also R67.1, R68.2; no longer D46.3 (K), R65.1, R66.2
- net MCU_supply_voltage_input: now also R59.1, R61.2; no longer D44.3 (K), R54.1, R55.2
- net RESISTIVE_SENSOR_0_190: now also R56.1
- new net: C32.1, D45.3 (K), R57.1, U6.3 (+)
- new net: C30.1, D44.3 (K), R54.1, R55.2, U6.5 (+)
- new net: C35.1, D46.3 (K), R65.1, R66.2, U6.10 (+)
- new net: R62.1, R63.2, U6.1
- new net: R60.2, R62.2, U6.2 (-)
- new net: R59.2, U6.6 (-), U6.7
- new net: R67.2, U6.8, U6.9 (-)
- no-connect marks 0 -> 3
Other:
- moved on the sheet: D44, D45, D46, R54, R55, R56, R57, R65, R66

Commit message: update pcb
Parts:
- added L4: FB, Inductor_SMD:L_1206_3216Metric_Pad1.42x1.75mm_HandSolder, symbol Device:L
Connections:
- net +5v_FROM_MCU: now also L4.1; no longer C29.1, R58.2
- new net: C29.1, L4.2, R58.2
Changed lines of the file:
@@
 Wire Wire Line
 	2650 1050 2850 1050
-Text GLabel 1850 1050 0    50   Input ~ 0
+Text GLabel 1300 1050 0    50   Input ~ 0
 +5v_FROM_MCU
 Wire Wire Line
@@
 Wire Wire Line
 	2350 1050 2200 1050
-Wire Wire Line
-	1850 1050 2200 1050
 Connection ~ 2200 1050
 Wire Wire Line
@@
 	1    0    0    -1
 $EndComp
+$Comp
+L Device:L L4
+U 1 1 607FD4F7
+P 1600 1050
+F 0 "L4" V 1419 1050 50  0000 C CNN
+F 1 "FB" V 1510 1050 50  0000 C CNN
+F 2 "Inductor_SMD:L_1206_3216Metric_Pad1.42x1.75mm_HandSolder" H 1600 1050 50  0001 C CNN
+F 3 "~" H 1600 1050 50  0001 C CNN
+	1    1600 1050
+	0    -1   -1   0
+$EndComp
+Wire Wire Line
+	1750 1050 2200 1050
+Wire Wire Line
+	1450 1050 1300 1050
 $EndSCHEMATC
