File: KiCad/Car_bs_controller_nex_mega/Analog_input.sch (KiCad schematic (older format))
At the start: 28 parts, among them U5 TL431DBZ, U6 MCP6004

Commit message: update
Parts:
- R56: value 1k -> 2k*
- R62: value 10k -> 10k*
- R64: value 10k -> 15k*
- U6: value MCP6004 -> MCP6004(LM324)
Other:
- note added: "15k(LM324)\n10k(MCP6004)"
- note added: "2.5V"
- note added: "k=1+(R62/R60)"
Changed lines of the file:
@@
 P 4500 3600
 F 0 "U6" H 4500 3967 50  0000 C CNN
-F 1 "MCP6004" H 4500 3876 50  0000 C CNN
+F 1 "MCP6004(LM324)" H 4500 3876 50  0000 C CNN
 F 2 "Package_SO:SOIC-14_3.9x8.7mm_P1.27mm" H 4450 3700 50  0001 C CNN
 F 3 "http://ww1.microchip.com/downloads/en/DeviceDoc/21733j.pdf" H 4550 3800 50  0001 C CNN
@@
 	1    2850 4100
 	1    0    0    -1
-$EndComp
-$Comp
-L Car_bs_controller_nex_mega-rescue:R-Device R?
-U 1 1 60104923
-P 1950 3050
-AR Path="/5FF96B9E/60104923" Ref="R?"  Part="1"
-AR Path="/60100EBE/60104923" Ref="R56"  Part="1"
-F 0 "R56" V 1743 3050 50  0000 C CNN
-F 1 "1k" V 1834 3050 50  0000 C CNN
-F 2 "Resistor_SMD:R_0805_2012Metric" V 1880 3050 50  0001 C CNN
-F 3 "~" H 1950 3050 50  0001 C CNN
-	1    1950 3050
-	-1   0    0    1
 $EndComp
 $Comp
@@
 AR Path="/60100EBE/60A64790" Ref="R62"  Part="1"
 F 0 "R62" V 4243 4050 50  0000 C CNN
-F 1 "10k" V 4334 4050 50  0000 C CNN
+F 1 "10k*" V 4334 4050 50  0000 C CNN
 F 2 "Resistor_SMD:R_0603_1608Metric_Pad0.98x0.95mm_HandSolder" V 4380 4050 50  0001 C CNN
 F 3 "~" H 4450 4050 50  0001 C CNN
@@
 AR Path="/60100EBE/60A78379" Ref="R64"  Part="1"
 F 0 "R64" V 5393 3900 50  0000 C CNN
-F 1 "10k" V 5484 3900 50  0000 C CNN
+F 1 "15k*" V 5484 3900 50  0000 C CNN
 F 2 "Resistor_SMD:R_0603_1608Metric_Pad0.98x0.95mm_HandSolder" V 5530 3900 50  0001 C CNN
 F 3 "~" H 5600 3900 50  0001 C CNN
@@
 P 3400 5950
 F 0 "U6" H 3400 6317 50  0000 C CNN
-F 1 "MCP6004" H 3400 6226 50  0000 C CNN
+F 1 "MCP6004(LM324)" H 3400 6226 50  0000 C CNN
 F 2 "Package_SO:SOIC-14_3.9x8.7mm_P1.27mm" H 3350 6050 50  0001 C CNN
 F 3 "http://ww1.microchip.com/downloads/en/DeviceDoc/21733j.pdf" H 3450 6150 50  0001 C CNN
@@
 P 8700 1800
 F 0 "U6" H 8700 2167 50  0000 C CNN
-F 1 "MCP6004" H 8700 2076 50  0000 C CNN
+F 1 "MCP6004(LM324)" H 8700 2076 50  0000 C CNN
 F 2 "Package_SO:SOIC-14_3.9x8.7mm_P1.27mm" H 8650 1900 50  0001 C CNN
 F 3 "http://ww1.microchip.com/downloads/en/DeviceDoc/21733j.pdf" H 8750 2000 50  0001 C CNN
@@
 P 7200 5250
 F 0 "U6" H 6800 5300 50  0000 L CNN
-F 1 "MCP6004" H 6650 5200 50  0000 L CNN
+F 1 "MCP6004(LM324)" H 6650 5200 50  0000 L CNN
 F 2 "Package_SO:SOIC-14_3.9x8.7mm_P1.27mm" H 7150 5350 50  0001 C CNN
 F 3 "http://ww1.microchip.com/downloads/en/DeviceDoc/21733j.pdf" H 7250 5450 50  0001 C CNN
@@
 P 9000 4050
 F 0 "U6" H 9000 4417 50  0000 C CNN
-F 1 "MCP6004" H 9000 4326 50  0000 C CNN
+F 1 "MCP6004(LM324)" H 9000 4326 50  0000 C CNN
 F 2 "Package_SO:SOIC-14_3.9x8.7mm_P1.27mm" H 8950 4150 50  0001 C CNN
 F 3 "http://ww1.microchip.com/downloads/en/DeviceDoc/21733j.pdf" H 9050 4250 50  0001 C CNN
@@
 Wire Wire Line
 	1450 1050 1300 1050
+$Comp
+L Car_bs_controller_nex_mega-rescue:R-Device R?
+U 1 1 60104923
+P 1950 3050
+AR Path="/5FF96B9E/60104923" Ref="R?"  Part="1"
+AR Path="/60100EBE/60104923" Ref="R56"  Part="1"
+F 0 "R56" V 1743 3050 50  0000 C CNN
+F 1 "2k*" V 1834 3050 50  0000 C CNN
+F 2 "Resistor_SMD:R_0805_2012Metric" V 1880 3050 50  0001 C CNN
+F 3 "~" H 1950 3050 50  0001 C CNN
+	1    1950 3050
+	-1   0    0    1
+$EndComp
+Text Notes 4000 3100 0    79   ~ 0
+k=1+(R62/R60)
+Text Notes 5900 3950 0    50   ~ 0
+15k(LM324)\n10k(MCP6004)
+Text Notes 5500 3550 0    50   ~ 0
+2.5V
 $EndSCHEMATC

Commit message: Changes
Other:
- note added: "Optional"
Changed lines of the file:
@@
 Text Notes 5500 3550 0    50   ~ 0
 2.5V
+Wire Notes Line
+	550  750  4700 750
+Wire Notes Line
+	4700 750  4700 1950
+Wire Notes Line
+	4700 1950 550  1950
+Wire Notes Line
+	550  1950 550  750
+Text Notes 800  1650 0    79   ~ 16
+Optional
 $EndSCHEMATC
