File: KiCad/Car_bs_controller_nex_mega/Car_bs_controller_nex_mega.sch (KiCad schematic (older format))
At the start: 0 parts

Commit message: Pcb and shematic changed
Changed lines of the file:
@@
 $EndSheet
 $Sheet
-S 4050 2650 1950 900
+S 3900 2650 1950 900
 U 5FF96CA3
 F0 "Links" 50
