File: KiCad/Car_bs_controller_nex_mega/Power supply.sch (KiCad schematic (older format))
At the start: 49 parts, among them U1 MP1584EN(SOIC8E), U2 MP1584EN(SOIC8E)

Commit message: big update
Parts:
- removed C1, C11, C13: 100n, Capacitor_SMD:C_0805_2012Metric, symbol Device:C
- removed C10, C12: 150p, Capacitor_SMD:C_0805_2012Metric, symbol Device:C
- removed C14: 22mk 10v, Capacitor_SMD:C_1812_4532Metric, symbol Device:C
- removed C16: 22mk 16v, Capacitor_SMD:C_1812_4532Metric, symbol Device:C
- removed C19: 100mk 25v, Capacitor_THT:CP_Radial_D8.0mm_P3.80mm, symbol Device:CP
- removed C2, C5: 100mk 50v, Capacitor_THT:CP_Radial_D8.0mm_P3.80mm, symbol Device:CP
- removed C3, C8: 10mk 50v, Capacitor_SMD:C_1812_4532Metric, symbol Device:C
- removed C9: 1n, Capacitor_SMD:C_0603_1608Metric, symbol Device:C
- removed D10, D9: SS34, Diode_SMD:D_SMB, symbol Device:D_Schottky
- removed D8: 5v6, Diode_SMD:D_MELF, symbol Device:D_Zener
- removed L2: 15uH, Inductor_SMD:L_7.3x7.3_H4.5, symbol Device:L
- removed R10, R12: 100k, Resistor_SMD:R_0805_2012Metric, symbol Device:R
- removed R11, R14: 30k, Resistor_SMD:R_0805_2012Metric, symbol Device:R
- removed R13: 160k, Resistor_SMD:R_0805_2012Metric, symbol Device:R
- removed R15: 240k, Resistor_SMD:R_0805_2012Metric, symbol Device:R
- removed R3: 100k, Resistor_SMD:R_0603_1608Metric, symbol Device:R
- removed R4: 30k, Resistor_SMD:R_0603_1608Metric, symbol Device:R
- removed R5: 24k, Resistor_SMD:R_0603_1608Metric, symbol Device:R
- removed R7, R9: 200k, Resistor_SMD:R_0805_2012Metric, symbol Device:R
- removed R8: 24k, Resistor_SMD:R_0805_2012Metric, symbol Device:R
- removed U1, U2: MP1584EN(SOIC8E), OLIMEX_IC-FP:SOIC-8-EP, symbol Car_bs_controller_nex_mega-rescue:MP1584EN(SOIC8E)-OLIMEX_IC
- added C1: 100n, Capacitor_SMD:C_0805_2012Metric, symbol Car_bs_controller_nex_mega-rescue:C-Device
- added C11, C13: 220mk 16v, Capacitor_THT:CP_Radial_D6.3mm_P2.50mm, symbol Car_bs_controller_nex_mega-rescue:CP-Device
- added C4: 10mk, Capacitor_SMD:C_1210_3225Metric_Pad1.33x2.70mm_HandSolder, symbol Car_bs_controller_nex_mega-rescue:C-Device
- added C7, C8, C9: 220mk 10v, Capacitor_THT:CP_Radial_D6.3mm_P2.50mm, symbol Car_bs_controller_nex_mega-rescue:CP-Device
- added D8: Cbc_power_module, Cbc_power_module:Cbc_power_module, symbol Cbc_power_module:Cbc_power_module
- added D9: SMBJ5CA, Diode_SMD:D_SMA, symbol Car_bs_controller_nex_mega-rescue:D_TVS-Device
- added R3: 1k, Resistor_SMD:R_0603_1608Metric_Pad0.98x0.95mm_HandSolder, symbol Car_bs_controller_nex_mega-rescue:R-Device
- added R4: 2k, Resistor_SMD:R_0603_1608Metric_Pad0.98x0.95mm_HandSolder, symbol Car_bs_controller_nex_mega-rescue:R-Device
- C10: renamed from C18; symbol Device:C -> Car_bs_controller_nex_mega-rescue:C-Device
- C12: renamed from C17; value 100mk 16v -> 220mk 16v; footprint Capacitor_THT:CP_Radial_D8.0mm_P3.80mm -> Capacitor_THT:CP_Radial_D6.3mm_P2.50mm; symbol Device:CP -> Car_bs_controller_nex_mega-rescue:CP-Device
- C2: renamed from C4; value 100mk 50v -> 220mk 25v; symbol Device:CP -> Car_bs_controller_nex_mega-rescue:CP-Device
- C3: renamed from C7; symbol Device:C -> Car_bs_controller_nex_mega-rescue:C-Device
- C5: renamed from C6; footprint Capacitor_SMD:C_0603_1608Metric -> Capacitor_SMD:C_0805_2012Metric; symbol Device:C -> Car_bs_controller_nex_mega-rescue:C-Device
- C6: renamed from C15; symbol Device:C -> Car_bs_controller_nex_mega-rescue:C-Device
- D1: renamed from D7; symbol Device:LED -> Car_bs_controller_nex_mega-rescue:LED-Device
- D2: renamed from D1; symbol Device:D_TVS -> Car_bs_controller_nex_mega-rescue:D_TVS-Device
- D3: renamed from D4; symbol Device:D_TVS -> Car_bs_controller_nex_mega-rescue:D_TVS-Device
- D4: renamed from D3; footprint Diode_SMD:D_SMC -> Diode_SMD:D_SMB; symbol Device:D -> Car_bs_controller_nex_mega-rescue:D-Device
- D5, D6: symbol Device:D -> Car_bs_controller_nex_mega-rescue:D-Device
- D7: renamed from D2; symbol Device:D -> Car_bs_controller_nex_mega-rescue:D-Device
- F1: symbol Device:Fuse -> Car_bs_controller_nex_mega-rescue:Fuse-Device
- L1: value 15uH -> 47uH
- R1: renamed from R6; footprint Resistor_SMD:R_0603_1608Metric -> Resistor_SMD:R_0603_1608Metric_Pad0.98x0.95mm_HandSolder; symbol Device:R -> Car_bs_controller_nex_mega-rescue:R-Device
- R2: renamed from R1; value 100R -> 2k; footprint Resistor_SMD:R_0805_2012Metric -> Resistor_SMD:R_0603_1608Metric_Pad0.98x0.95mm_HandSolder; symbol Device:R -> Car_bs_controller_nex_mega-rescue:R-Device
- R5: renamed from R2; value 30k -> 2k; footprint Resistor_SMD:R_0603_1608Metric -> Resistor_SMD:R_0603_1608Metric_Pad0.98x0.95mm_HandSolder; symbol Device:R -> Car_bs_controller_nex_mega-rescue:R-Device
Connections:
- net +12V: now also R1.2, C1.1
- net 5V_sensors_stab: now also C7.1, C8.1, C9.1, D8.9 (OUT_5v), D9.1 (A1); no longer C12.1, L1.2
- net 7.2V_stab: now also C12.1, C11.1, C13.1, D8.6 (OUT_7.2v)
- net GND: now also C1.2, C11.2, C13.2, C4.2, C7.2, C8.2, C9.2, D8.1 (GND), D8.7 (GND), D8.8 (GND), D9.2 (A2), R3.2
- net MCU_5V_sensors_enable: now also R5.1; no longer D7.2 (A)
- net MCU_main_supply_enable: now also R4.1; no longer D5.2 (A)
- net at C2.1, C3.1: now also L1.2, D8.2 (IN1), D8.3 (IN2); no longer D4.1 (K), R1.2
- net at D5.1 (K): now also D6.1 (K), C4.1, D8.4 (EN1)
- net at L1.1: now also D4.1 (K)
- net at C5.1: now also D7.1 (K), D8.5 (EN2); no longer R5.2
- net at D3.1 (A1), D6.2 (A), R2.2: now also R3.1
- new net: D7.2 (A), R5.2
- new net: D5.2 (A), R4.2
Other:
- note removed: "Vout=(0.8*(R13+R11))/R11\nVout=(0.8*(160+30))/30=5.067V"
- note removed: "Vout=(0.8*(R15+R14))/R14\nVout=(0.8*(240+30))/30=7.2V"
- moved on the sheet: C10, C12, C2, C3, C5, C6, D1, D2, D3, D4, D5, D6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
