File: KiCad/Car_bs_controller_nex_mega/Car_bs_controller_nex_mega.kicad_pcb (KiCad board)
At the start: 2 copper layers, 99.5 x 83 mm, 205 parts, among them J1 Power, J10 Encoder, J11 LCD_Nextion, J12 PUMP_RELAY, J13 LIGHT_RELAY, J14 LIGHT_RELAY, J15 I2C, J2 Inputs, J3 Proxy, J4 PJON, J5 RS485, J6 RES_SENS, J7 1_WARE, J8 Outputs, J9 LCD_ST7920, K1 1393217-4, K2 1393217-4, K3 1393217-4, Q1 BSS138, Q2 BC857, SW1 SW_Push, U1 MP1584EN(SOIC8E), U2 MP1584EN(SOIC8E), U3 MEGA_PRO_EMBED_CH340G___ATMEG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, U4 ADM705, U5 MAX485E, U6 ULN2003A, U7 TL431DBZ

Commit message: Update
Parts:
- J14: value LIGHT_RELAY -> CONVERTER_RELAY
Connections:
- U3 pad A10: (no net) -> Net-(U3-PadA10)
- U3 pad A11: (no net) -> Net-(U3-PadA11)
- U3 pad A12: (no net) -> Net-(U3-PadA12)
- U3 pad A13: (no net) -> Net-(U3-PadA13)
- U3 pad A14: (no net) -> Net-(U3-PadA14)
- U3 pad A15: (no net) -> Net-(U3-PadA15)
- U3 pad A7: (no net) -> Net-(U3-PadA7)
- U3 pad A8: (no net) -> Net-(U3-PadA8)
- U3 pad A9: (no net) -> Net-(U3-PadA9)
- U3 pad D11: (no net) -> Net-(U3-PadD11)
- U3 pad D12: (no net) -> Net-(U3-PadD12)
- U3 pad D14: (no net) -> Net-(U3-PadD14)
- U3 pad D15: (no net) -> Net-(U3-PadD15)
- U3 pad D25: (no net) -> Net-(U3-PadD25)
- U3 pad D26: (no net) -> Net-(U3-PadD26)
- U3 pad D27: (no net) -> Net-(U3-PadD27)
- U3 pad D28: (no net) -> Net-(U3-PadD28)
- U3 pad D29: (no net) -> Net-(U3-PadD29)
- U3 pad D30: (no net) -> Net-(U3-PadD30)
- U3 pad D38: (no net) -> Net-(U3-PadD38)
- U3 pad D39: (no net) -> Net-(U3-PadD39)
- U3 pad D40: (no net) -> Net-(U3-PadD40)
- U3 pad D45: (no net) -> Net-(U3-PadD45)
- U3 pad D46: (no net) -> Net-(U3-PadD46)
- U3 pad D47: (no net) -> Net-(U3-PadD47)
- U3 pad D48: (no net) -> Net-(U3-PadD48)
- U3 pad D49: (no net) -> Net-(U3-PadD49)
- U3 pad D50: (no net) -> Net-(U3-PadD50)
- U3 pad MISO: (no net) -> Net-(U3-PadMISO)
- U3 pad MOSI: (no net) -> Net-(U3-PadMOSI)
- U3 pad RESET: (no net) -> Net-(U3-PadRESET)
- U3 pad RX: (no net) -> Net-(U3-PadRX)
- U3 pad SCK: (no net) -> Net-(U3-PadSCK)
- U3 pad TX: (no net) -> Net-(U3-PadTX)

Commit message: big update
Parts:
- removed the C10 at (81.3, 81.8)
- removed the C12 at (79.9, 62.9)
- removed the C14 at (83.4, 87.3)
- removed the C16 at (88.8, 70.8)
- removed the C19 at (93.4, 72.7)
- removed the C2 at (65.3, 68.2)
- removed the C27 at (152.2, 91.4)
- removed the C3 at (92.4, 87.5)
- removed the C5 at (70.4, 74.4)
- removed the D10 at (89.6, 61.9)
- removed the D11 at (98.8, 59.4)
- removed the D12 at (94.5, 59.3)
- removed the D13 at (99.9, 59.4)
- removed the D14 at (107.6, 59.5)
- removed the D15 at (94.8, 59.4)
- removed the D16 at (103.3, 59.4)
- removed the D46 at (149.4, 104.2)
- removed D48, D50: 2v4, Diode_SMD:D_MELF
- removed the F2 at (135.9, 57.3)
- removed the F3 at (116.1, 58.0)
- removed K1, K2, K3: 1393217-4, RELAY_1393217-4
- removed the R10 at (85.5, 81.7)
- removed the R11 at (85.8, 79.4)
- removed the R12 at (83.6, 62.8)
- removed the R13 at (81.1, 78.6)
- removed the R14 at (79.8, 60.1)
- removed the R15 at (87.4, 58.0)
- removed the R16 at (89.7, 48.7)
- removed the R17 at (85.9, 48.7)
- removed the R18 at (101.3, 48.7)
- removed the R19 at (112.3, 48.6)
- removed the R20 at (97.4, 48.7)
- removed the R21 at (93.6, 48.7)
- removed the R42 at (123.2, 56.9)
- removed the R43 at (140.3, 64.4)
- removed the R5 at (78.5, 87.4)
- removed the R7 at (91.6, 82.3)
- removed R70, R73, R76: 2k2, Resistor_SMD:R_0805_2012Metric
- removed the R8 at (73.9, 62.9)
- removed the R9 at (93.4, 64.4)
- removed the U1 at (84.2, 83.9)
- removed the U2 at (87.2, 62.1)
- added C20: 220mk 10v, Capacitor_THT:CP_Radial_D6.3mm_P2.50mm, F.Cu at (138.4, 84.1)
- added C21: 10mk, Capacitor_Tantalum_SMD:CP_EIA-7343-15_Kemet-W_Pad2.25x2.55mm_HandSolder, B.Cu at (149.6, 95.6)
- added C23: 1n, Resistor_SMD:R_0603_1608Metric_Pad0.98x0.95mm_HandSolder, B.Cu at (143.9, 92.9)
- added C30: 10n, Resistor_SMD:R_0603_1608Metric, B.Cu at (116.2, 81.9)
- added C32: 10n, Resistor_SMD:R_0603_1608Metric, B.Cu at (112.8, 87.9)
- added C33: 100n, Resistor_SMD:R_0603_1608Metric, B.Cu at (124.3, 91.4)
- added C34: 10mk, Capacitor_Tantalum_SMD:CP_EIA-6032-15_Kemet-U, B.Cu at (124.6, 78.7)
- added C35: 10n, Resistor_SMD:R_0603_1608Metric, B.Cu at (130.3, 88.0)
- added C4: 10mk, Capacitor_SMD:C_1210_3225Metric_Pad1.33x2.70mm_HandSolder, F.Cu at (62.1, 87.9)
- added C7: 220mk 10v, Capacitor_THT:CP_Radial_D6.3mm_P2.50mm, F.Cu at (91.9, 86.4)
- added D22: BAV99, Package_TO_SOT_SMD:SOT-23, B.Cu at (173.4, 73.8)
- added D23: BAV99, Package_TO_SOT_SMD:SOT-23, B.Cu at (183.4, 63.8)
- added D24: BAV99, Package_TO_SOT_SMD:SOT-23, F.Cu at (149.2, 105.9)
- added D25: BAV99, Package_TO_SOT_SMD:SOT-23, B.Cu at (187.4, 69.2)
- added D26: BAV99, Package_TO_SOT_SMD:SOT-23, B.Cu at (182.4, 74.8)
- added D27: BAV99, Package_TO_SOT_SMD:SOT-23, B.Cu at (196.4, 69.8)
- added JP1: SolderJumper_2_Open, Jumper:SolderJumper-2_P1.3mm_Open_RoundedPad1.0x1.5mm, B.Cu at (144.1, 83.6)
- added L3: BLN, Inductor_SMD:L_0805_2012Metric_Pad1.15x1.40mm_HandSolder, F.Cu at (167.2, 67.4)
- added R27: 1k, Resistor_SMD:R_0603_1608Metric_Pad0.98x0.95mm_HandSolder, B.Cu at (145.7, 89.4)
- added R28: 220R, Resistor_SMD:R_0603_1608Metric_Pad0.98x0.95mm_HandSolder, B.Cu at (152.1, 83.4)
- added R38: 470R, Resistor_SMD:R_0603_1608Metric_Pad0.98x0.95mm_HandSolder, F.Cu at (161.4, 69.5)
- added R45: 1k, Resistor_SMD:R_0805_2012Metric_Pad1.20x1.40mm_HandSolder, F.Cu at (126.5, 85.5)
- added R59: 6k8, Resistor_SMD:R_0603_1608Metric_Pad0.98x0.95mm_HandSolder, B.Cu at (119.2, 80.6)
- added R61: 10k, Resistor_SMD:R_0603_1608Metric_Pad0.98x0.95mm_HandSolder, B.Cu at (116.0, 79.8)
- added R62: 10k, Resistor_SMD:R_0603_1608Metric_Pad0.98x0.95mm_HandSolder, B.Cu at (118.5, 88.8)
- added R63: 6k8, Resistor_SMD:R_0603_1608Metric_Pad0.98x0.95mm_HandSolder, B.Cu at (120.2, 91.9)
- added R64: 10k, Resistor_SMD:R_0603_1608Metric_Pad0.98x0.95mm_HandSolder, B.Cu at (116.4, 92.0)
- added R67: 6k8, Resistor_SMD:R_0603_1608Metric_Pad0.98x0.95mm_HandSolder, B.Cu at (130.5, 81.8)
- added R68: 10k, Resistor_SMD:R_0603_1608Metric_Pad0.98x0.95mm_HandSolder, B.Cu at (130.9, 78.8)
- added REL1: SRA-12VDC-CL, ab2_relay:AB2_SRA-12VDC-CL, B.Cu at (81.4, 102.4)
- added REL2: SRA-12VDC-CL, ab2_relay:AB2_SRA-12VDC-CL, B.Cu at (95.1, 102.4)
- added REL3: SRA-12VDC-CL, ab2_relay:AB2_SRA-12VDC-CL, B.Cu at (67.7, 99.1)
- added U6: MCP6004, Package_SO:SOIC-14_3.9x8.7mm_P1.27mm, B.Cu at (124.3, 85.8)
- C11, C13: value 100n -> 220mk 16v; footprint Capacitor_SMD:C_0805_2012Metric -> Capacitor_THT:CP_Radial_D6.3mm_P2.50mm; moved to F.Cu
- C12: renamed from C17; value 100mk 16v -> 220mk 16v; footprint Capacitor_THT:CP_Radial_D8.0mm_P3.80mm -> Capacitor_THT:CP_Radial_D6.3mm_P2.50mm
- C14: renamed from C20; footprint Capacitor_SMD:C_0805_2012Metric -> Capacitor_SMD:C_0603_1608Metric_Pad1.08x0.95mm_HandSolder
- C15: renamed from C21; footprint Capacitor_SMD:C_0805_2012Metric -> Capacitor_SMD:C_0603_1608Metric_Pad1.08x0.95mm_HandSolder
- C16: renamed from C22; footprint Capacitor_SMD:C_0805_2012Metric -> Capacitor_SMD:C_0603_1608Metric_Pad1.08x0.95mm_HandSolder
- C17: renamed from C23; footprint Capacitor_SMD:C_0805_2012Metric -> Capacitor_SMD:C_0603_1608Metric_Pad1.08x0.95mm_HandSolder
- C18: renamed from C24; footprint Capacitor_SMD:C_0805_2012Metric -> Capacitor_SMD:C_0603_1608Metric_Pad1.08x0.95mm_HandSolder
- C19: renamed from C25; footprint Capacitor_SMD:C_0805_2012Metric -> Capacitor_SMD:C_0603_1608Metric_Pad1.08x0.95mm_HandSolder
- C2: renamed from C4; value 100mk 50v -> 220mk 25v
- C24: renamed from C28; value 4m7 -> 10m; footprint Capacitor_SMD:C_1206_3216Metric -> Capacitor_SMD:C_1210_3225Metric_Pad1.33x2.70mm_HandSolder
- C25: renamed from C29; footprint Capacitor_SMD:C_0805_2012Metric -> Capacitor_SMD:C_0603_1608Metric_Pad1.08x0.95mm_HandSolder
- C28: renamed from C32; moved to F.Cu
- C5: renamed from C6; footprint Capacitor_SMD:C_0603_1608Metric -> Capacitor_SMD:C_0805_2012Metric; moved to F.Cu
- C6: renamed from C15; moved to B.Cu
- C8: value 10mk 50v -> 220mk 10v; footprint Capacitor_SMD:C_1812_4532Metric -> Capacitor_THT:CP_Radial_D6.3mm_P2.50mm; moved to F.Cu
- C9: value 1n -> 220mk 10v; footprint Capacitor_SMD:C_0603_1608Metric -> Capacitor_THT:CP_Radial_D6.3mm_P2.50mm; moved to F.Cu
- D2: renamed from D1; moved to F.Cu
- D28: renamed from D29; moved to F.Cu
- D4: renamed from D3; footprint Diode_SMD:D_SMC -> Diode_SMD:D_SMB
- D5, D6: moved to F.Cu
- D7: renamed from D2; moved to F.Cu
- D8: value 5v6 -> Cbc_power_module; footprint Diode_SMD:D_MELF -> Cbc_power_module:Cbc_power_module; moved to F.Cu
- D9: value SS34 -> SMBJ5CA; footprint Diode_SMD:D_SMB -> Diode_SMD:D_SMA
- F2: renamed from F5; footprint Fuse:Fuse_1210_3225Metric -> Fuse:Fuse_1206_3216Metric_Pad1.42x1.75mm_HandSolder
- F3: renamed from F6; footprint Fuse:Fuse_1210_3225Metric -> Fuse:Fuse_1206_3216Metric_Pad1.42x1.75mm_HandSolder
- F4: value 200mA -> 200mA 5v; footprint Fuse:Fuse_1210_3225Metric -> Fuse:Fuse_1206_3216Metric_Pad1.42x1.75mm_HandSolder
- L1: value 15uH -> 47uH
- L2: value 15uH -> BLN; footprint Inductor_SMD:L_7.3x7.3_H4.5 -> Inductor_SMD:L_0805_2012Metric_Pad1.15x1.40mm_HandSolder
- R1: renamed from R6; footprint Resistor_SMD:R_0603_1608Metric -> Resistor_SMD:R_0603_1608Metric_Pad0.98x0.95mm_HandSolder; moved to F.Cu
- R10: renamed from R26; footprint Resistor_SMD:R_0805_2012Metric -> Resistor_SMD:R_0603_1608Metric_Pad0.98x0.95mm_HandSolder
- R11: renamed from R27; footprint Resistor_SMD:R_0805_2012Metric -> Resistor_SMD:R_0603_1608Metric_Pad0.98x0.95mm_HandSolder
- R12: renamed from R28; footprint Resistor_SMD:R_0805_2012Metric -> Resistor_SMD:R_0603_1608Metric_Pad0.98x0.95mm_HandSolder
- R13: renamed from R29; footprint Resistor_SMD:R_0805_2012Metric -> Resistor_SMD:R_0603_1608Metric_Pad0.98x0.95mm_HandSolder
- R14: renamed from R30; footprint Resistor_SMD:R_0805_2012Metric -> Resistor_SMD:R_0603_1608Metric_Pad0.98x0.95mm_HandSolder
- R15: renamed from R31; footprint Resistor_SMD:R_0805_2012Metric -> Resistor_SMD:R_0603_1608Metric_Pad0.98x0.95mm_HandSolder
- R16: renamed from R32; footprint Resistor_SMD:R_0805_2012Metric -> Resistor_SMD:R_0603_1608Metric_Pad0.98x0.95mm_HandSolder
- R17: renamed from R33; footprint Resistor_SMD:R_0805_2012Metric -> Resistor_SMD:R_0603_1608Metric_Pad0.98x0.95mm_HandSolder
- R2: renamed from R1; value 100R -> 2k; footprint Resistor_SMD:R_0805_2012Metric -> Resistor_SMD:R_0603_1608Metric_Pad0.98x0.95mm_HandSolder
- R21: renamed from R37; footprint Resistor_SMD:R_0603_1608Metric -> Resistor_SMD:R_0603_1608Metric_Pad0.98x0.95mm_HandSolder; moved to B.Cu
- R22: renamed from R40; footprint Resistor_SMD:R_0603_1608Metric -> Resistor_SMD:R_0603_1608Metric_Pad0.98x0.95mm_HandSolder
- R23: renamed from R38; footprint Resistor_SMD:R_0805_2012Metric -> Resistor_SMD:R_0603_1608Metric_Pad0.98x0.95mm_HandSolder; moved to F.Cu
- R25: renamed from R39; moved to B.Cu
- R26: renamed from R44; footprint Resistor_SMD:R_0603_1608Metric -> Resistor_SMD:R_0603_1608Metric_Pad0.98x0.95mm_HandSolder
- R29: renamed from R45; footprint Resistor_SMD:R_0603_1608Metric -> Resistor_SMD:R_0603_1608Metric_Pad0.98x0.95mm_HandSolder
- R3: value 100k -> 1k; footprint Resistor_SMD:R_0603_1608Metric -> Resistor_SMD:R_0603_1608Metric_Pad0.98x0.95mm_HandSolder
- R30: renamed from R46; footprint Resistor_SMD:R_0603_1608Metric -> Resistor_SMD:R_0603_1608Metric_Pad0.98x0.95mm_HandSolder
- R31: renamed from R48; footprint Resistor_SMD:R_0805_2012Metric -> Resistor_SMD:R_0603_1608Metric_Pad0.98x0.95mm_HandSolder
- R32: renamed from R47; value 2k2 -> 1k2
- R33: renamed from R49; footprint Resistor_SMD:R_0805_2012Metric -> Resistor_SMD:R_0603_1608Metric_Pad0.98x0.95mm_HandSolder
- R34: renamed from R50; value 2k2 -> 1k
- R35: renamed from R51; footprint Resistor_SMD:R_0805_2012Metric -> Resistor_SMD:R_0603_1608Metric_Pad0.98x0.95mm_HandSolder
- R36: renamed from R52; value 2k2 -> 1k
- R37: renamed from R53; footprint Resistor_SMD:R_0603_1608Metric -> Resistor_SMD:R_0603_1608Metric_Pad0.98x0.95mm_HandSolder
- R39: renamed from R54; footprint Resistor_SMD:R_0805_2012Metric -> Resistor_SMD:R_0603_1608Metric_Pad0.98x0.95mm_HandSolder
- R4: value 30k -> 2k; footprint Resistor_SMD:R_0603_1608Metric -> Resistor_SMD:R_0603_1608Metric_Pad0.98x0.95mm_HandSolder; moved to F.Cu
- R40: renamed from R55; footprint Resistor_SMD:R_0603_1608Metric -> Resistor_SMD:R_0603_1608Metric_Pad0.98x0.95mm_HandSolder
- R42: renamed from R57; footprint Resistor_SMD:R_0805_2012Metric -> Resistor_SMD:R_0603_1608Metric_Pad0.98x0.95mm_HandSolder
- R46: renamed from R61; value 2k2 -> 10k
- R47: renamed from R62; value 2k2 -> 10k
- R48: renamed from R63; value 2k2 -> 10k
- R49: renamed from R64; footprint Resistor_SMD:R_0805_2012Metric -> Resistor_SMD:R_0603_1608Metric_Pad0.98x0.95mm_HandSolder
- R5: renamed from R2; value 30k -> 2k; footprint Resistor_SMD:R_0603_1608Metric -> Resistor_SMD:R_0603_1608Metric_Pad0.98x0.95mm_HandSolder; moved to F.Cu
- R50: renamed from R65; footprint Resistor_SMD:R_0603_1608Metric -> Resistor_SMD:R_0603_1608Metric_Pad0.98x0.95mm_HandSolder
- R52: renamed from R77; moved to B.Cu
- R54: renamed from R67; value 10k -> 39k; footprint Resistor_SMD:R_0805_2012Metric -> Resistor_SMD:R_0603_1608Metric_Pad0.98x0.95mm_HandSolder
- R55: renamed from R68; value 1k -> 10k; footprint Resistor_SMD:R_0805_2012Metric -> Resistor_SMD:R_0603_1608Metric_Pad0.98x0.95mm_HandSolder
- R56: renamed from R72; value 2k2 -> 1k
- R57: renamed from R71; value 100R -> 10k; footprint Resistor_SMD:R_0805_2012Metric -> Resistor_SMD:R_0603_1608Metric_Pad0.98x0.95mm_HandSolder
- R58: renamed from R69; value 150R -> 330R
- R6: renamed from R22; footprint Resistor_SMD:R_0805_2012Metric -> Resistor_SMD:R_0603_1608Metric_Pad0.98x0.95mm_HandSolder
- R60: value 120R -> 2k2; footprint Resistor_SMD:R_1206_3216Metric -> Resistor_SMD:R_0603_1608Metric_Pad0.98x0.95mm_HandSolder
- R65: renamed from R74; value 10k -> 22k; footprint Resistor_SMD:R_0805_2012Metric -> Resistor_SMD:R_0603_1608Metric_Pad0.98x0.95mm_HandSolder
- R66: renamed from R75; value 1k -> 10k; footprint Resistor_SMD:R_0805_2012Metric -> Resistor_SMD:R_0603_1608Metric_Pad0.98x0.95mm_HandSolder
- R7: renamed from R23; value 22k -> 15k; footprint Resistor_SMD:R_0805_2012Metric -> Resistor_SMD:R_0603_1608Metric_Pad0.98x0.95mm_HandSolder
- R8: renamed from R24; footprint Resistor_SMD:R_0805_2012Metric -> Resistor_SMD:R_0603_1608Metric_Pad0.98x0.95mm_HandSolder
- R9: renamed from R25; value 22k -> 15k; footprint Resistor_SMD:R_0805_2012Metric -> Resistor_SMD:R_0603_1608Metric_Pad0.98x0.95mm_HandSolder
- moved L2 123.8 mm to (206.7, 60.1), turned to 0 degrees
- moved SW1 103.3 mm to (153.7, 54.8)
- moved R21 97.2 mm to (60.8, 49.7)
- moved R55 95.7 mm to (65.0, 47.9), turned to 180 degrees
- moved R54 92.1 mm to (65.0, 50.8), turned to 270 degrees
- moved D21 63.3 mm to (212.9, 62.1)
- moved D5 62.5 mm to (68.9, 77.0)
- moved C14 57.4 mm to (190.1, 64.4)
- moved D12 57.4 mm to (177.9, 74.2)
- moved D15 57.4 mm to (200.8, 61.8)
- moved D16 57.4 mm to (195.5, 65.4)
- moved D18 57.4 mm to (181.9, 79.3)
- moved D19 57.4 mm to (199.2, 78.8)
- moved R12 57.4 mm to (193.6, 73.4)
- moved R13 57.4 mm to (202.0, 67.0)
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- renumbered C18 to C10, C26 to C22, C30 to C26, C31 to C27, C33 to C29, C7 to C3, C34 to C31, D7 to D1, D17 to D10, D18 to D11, D19 to D12, D20 to D13, D21 to D14, D22 to D15, D23 to D16, D24 to D17, D25 to D18, D26 to D19, D27 to D20, D28 to D21, D30 to D29, D4 to D3, D32 to D30, D33 to D32, D34 to D33, D35 to D34, D36 to D35, D37 to D36, D38 to D37, D39 to D38, D40 to D39, D41 to D40, D42 to D41, D43 to D42, D44 to D43, D45 to D44, D47 to D45, D49 to D46, J15 to J12, J12 to J13, J13 to J14, J14 to J15, JP1 to JP2, R34 to R18, R35 to R19, R36 to R20, R41 to R24, R56 to R41, R58 to R43, R59 to R44, R66 to R51, R78 to R53, U3 to U1, U4 to U2, U5 to U3, U6 to U4, U7 to U5
Connections:
- C1 pad 1: Net-(C1-Pad1) -> +12V
- C11 pad 1: Net-(C11-Pad1) -> 7.2V_stab
- C11 pad 2: Net-(C11-Pad2) -> GND
- C12 pad 1: 5V_sensors_stab -> 7.2V_stab
- C13 pad 1: Net-(C13-Pad1) -> 7.2V_stab
- C13 pad 2: Net-(C13-Pad2) -> GND
- C2 pad 1: Net-(C1-Pad1) -> Net-(C2-Pad1)
- C24 pad 1: 5V_sensors_stab -> +5v_FROM_MCU
- C25 pad 1: 5V_sensors_stab -> +5v_FROM_MCU
- C3 pad 1: Net-(C1-Pad1) -> Net-(C2-Pad1)
- C5 pad 1: Net-(C6-Pad1) -> Net-(C5-Pad1)
- C8 pad 1: Net-(C1-Pad1) -> 5V_sensors_stab
- C9 pad 1: Net-(C9-Pad1) -> 5V_sensors_stab
- D10 pad 1: Net-(D11-Pad1) (its old number) -> WATER_FLOW_SENSOR_INPUT
- D11 pad 2: Net-(D12-Pad1) (its old number) -> SPARE_INPUT_1
- D12 pad 2: Net-(D15-Pad1) -> IGNITION_SWITCH_INPUT
- D13 pad 1: Net-(D13-Pad1) -> DOOR_SWITCH_INPUT
- D14 pad 1: Net-(D14-Pad1) -> PROXIMITY_SENSOR_INPUT
- D15 pad 1: Net-(D16-Pad1) -> LOW_WASHER_WATER_LEVEL_INPUT
- D28 pad 3: Net-(D29-Pad3) -> MCU_one_wire_PIN
- D29 pad 3: Net-(D30-Pad3) -> MCU_pjon_bus_PIN
- D3 pad 1: Net-(D4-Pad1) -> Net-(D3-Pad1)
- D33 pad 2: 5V_sensors_stab -> +5v_FROM_MCU
- D34 pad 2: 5V_sensors_stab -> +5v_FROM_MCU
- D4 pad 1: Net-(C1-Pad1) -> Net-(D4-Pad1)
- D41 pad 2: Net-(D42-Pad2) -> Net-(D41-Pad2)
- D42 pad 2: Net-(D43-Pad2) -> Net-(D42-Pad2)
- D43 pad 2: Net-(D44-Pad2) -> Net-(D43-Pad2)
- D44 pad 2: Net-(D45-Pad2) -> +5v_FROM_MCU
- D44 pad 3: MCU_supply_voltage_input -> Net-(C30-Pad1)
- D45 pad 2: Net-(D47-Pad2) -> +5v_FROM_MCU
- D45 pad 3: MCU_resistive_sensor_0_190 -> Net-(C32-Pad1)
- D46 pad 2: Net-(D49-Pad2) -> +5v_FROM_MCU
- D46 pad 3: MCU_sensors_voltage_test_input -> Net-(C35-Pad1)
- D5 pad 1: Net-(D5-Pad1) -> Net-(C4-Pad1)
- D5 pad 2: MCU_main_supply_enable -> Net-(D5-Pad2)
- D6 pad 1: Net-(D6-Pad1) -> Net-(C4-Pad1)
- D6 pad 2: Net-(D4-Pad1) -> Net-(D3-Pad1)
- D7 pad 1: Net-(D2-Pad1) -> Net-(C5-Pad1)
- D7 pad 2: MCU_5V_sensors_enable -> Net-(D7-Pad2)
- D8 pad 1: Net-(C9-Pad1) -> GND
- D8 pad 2: GND -> Net-(C2-Pad1)
- D9 pad 1: Net-(C11-Pad2) -> 5V_sensors_stab
- F4 pad 2: Net-(D44-Pad2) -> +5v_FROM_MCU
- J12 pad 1: +5v_FROM_MCU -> Net-(F4-Pad1)
- J13 pad 1: PUMP_RELAY_COM -> PUMP_RELAY_NO
- J13 pad 2: PUMP_RELAY_NO -> PUMP_RELAY_COM
- J14 pad 1: LIGHT_RELAY_COM -> LIGHT_RELAY_NO
- J14 pad 2: LIGHT_RELAY_NO -> LIGHT_RELAY_COM
- J15 pad 1: CONVERTER_RELAY_COM -> CONVERTER_RELAY_NO
- J15 pad 2: CONVERTER_RELAY_NO -> CONVERTER_RELAY_COM
- J3 pad 1: Net-(F3-Pad1) (its old number) -> Net-(D42-Pad2)
- J4 pad 1: Net-(F2-Pad1) (its old number) -> Net-(D41-Pad2)
- J7 pad 1: Net-(F4-Pad1) -> Net-(D43-Pad2)
- L1 pad 1: Net-(C11-Pad2) -> Net-(D4-Pad1)
- L1 pad 2: 5V_sensors_stab -> Net-(C2-Pad1)
- L2 pad 1: Net-(C13-Pad2) -> Net-(L2-Pad1)
- L2 pad 2: 7.2V_stab -> MCU_one_wire_PIN
- R1 pad 2: Net-(C1-Pad1) -> +12V
- R19 pad 1: Net-(D29-Pad3) -> Net-(L2-Pad1)
- R2 pad 2: Net-(D4-Pad1) -> Net-(D3-Pad1)
- R20 pad 1: Net-(D30-Pad3) -> Net-(L3-Pad1)
- R23 pad 2: Net-(D29-Pad3) -> MCU_one_wire_PIN
- R24 pad 2: Net-(D29-Pad3) -> MCU_one_wire_PIN
- R25 pad 1: Net-(D30-Pad3) -> MCU_pjon_bus_PIN
- R3 pad 1: Net-(D6-Pad1) -> Net-(D3-Pad1)
- R3 pad 2: Net-(C9-Pad1) -> GND
- R31 pad 1: 5V_sensors_stab -> +5v_FROM_MCU
- R33 pad 1: 5V_sensors_stab -> +5v_FROM_MCU
- R35 pad 1: 5V_sensors_stab -> +5v_FROM_MCU
- R4 pad 1: Net-(D5-Pad1) -> MCU_main_supply_enable
- R4 pad 2: Net-(C9-Pad1) -> Net-(D5-Pad2)
- R42 pad 1: 5V_sensors_stab -> +5v_FROM_MCU
- R5 pad 1: Net-(D2-Pad1) -> MCU_5V_sensors_enable
- R5 pad 2: Net-(C6-Pad1) -> Net-(D7-Pad2)
- R52 pad 2: +5v_FROM_MCU -> Net-(F4-Pad1)
- R53 pad 2: +5v_FROM_MCU -> Net-(F4-Pad1)
- R54 pad 1: MCU_supply_voltage_input -> Net-(C30-Pad1)
- R55 pad 2: MCU_supply_voltage_input -> Net-(C30-Pad1)
- R56 pad 1: Net-(D47-Pad2) -> RESISTIVE_SENSOR_0_190
- R57 pad 1: MCU_resistive_sensor_0_190 -> Net-(C32-Pad1)
- R60 pad 1: RS485_B -> GND
- R60 pad 2: RS485_A -> Net-(R60-Pad2)
- R65 pad 1: MCU_sensors_voltage_test_input -> Net-(C35-Pad1)
- R66 pad 2: MCU_sensors_voltage_test_input -> Net-(C35-Pad1)
- SW1 pad 1: MCU_button_on_board -> Net-(R38-Pad1)
- U1 pad A10: Net-(U3-PadA10) -> (no net)
- U1 pad A11: Net-(U3-PadA11) -> (no net)
- U1 pad A12: Net-(U3-PadA12) -> (no net)
- U1 pad A13: Net-(U3-PadA13) -> (no net)
- U1 pad A14: Net-(U3-PadA14) -> (no net)
- U1 pad A15: Net-(U3-PadA15) -> (no net)
- U1 pad A7: Net-(U3-PadA7) -> (no net)
- U1 pad A8: Net-(U3-PadA8) -> (no net)
- U1 pad A9: Net-(U3-PadA9) -> (no net)
- U1 pad D11: Net-(U3-PadD11) -> (no net)
- U1 pad D12: Net-(U3-PadD12) -> (no net)
- U1 pad D14: Net-(U3-PadD14) -> (no net)
- U1 pad D15: Net-(U3-PadD15) -> (no net)
- U1 pad D25: Net-(U3-PadD25) -> (no net)
- U1 pad D26: Net-(U3-PadD26) -> (no net)
- U1 pad D27: Net-(U3-PadD27) -> (no net)
- U1 pad D28: Net-(U3-PadD28) -> (no net)
- U1 pad D29: Net-(U3-PadD29) -> (no net)
- U1 pad D30: Net-(U3-PadD30) -> (no net)
- U1 pad D38: Net-(U3-PadD38) -> (no net)
- U1 pad D39: Net-(U3-PadD39) -> (no net)
- U1 pad D40: Net-(U3-PadD40) -> (no net)
- U1 pad D45: Net-(U3-PadD45) -> (no net)
- U1 pad D46: Net-(U3-PadD46) -> (no net)
- U1 pad D47: Net-(U3-PadD47) -> (no net)
- U1 pad D48: Net-(U3-PadD48) -> (no net)
- U1 pad D49: Net-(U3-PadD49) -> (no net)
- U1 pad D50: Net-(U3-PadD50) -> (no net)
- U1 pad MISO: Net-(U3-PadMISO) -> (no net)
- U1 pad MOSI: Net-(U3-PadMOSI) -> (no net)
- U1 pad RESET: Net-(U3-PadRESET) -> (no net)
- U1 pad RX: Net-(U3-PadRX) -> (no net)
- U1 pad SCK: Net-(U3-PadSCK) -> (no net)
- U1 pad TX: Net-(U3-PadTX) -> (no net)
- U2 pad 7: MCU_rst -> Net-(R28-Pad2)
- U3 pad 8: 5V_sensors_stab -> +5v_FROM_MCU
Routing:
- net GND: track 785.2 -> 404.0 mm, vias 8 -> 5
- net 5V_sensors_stab: track 407.4 -> 146.5 mm, vias 5 -> 0
- net +5v_FROM_MCU: track 250.2 -> 55.3 mm, vias 9 -> 2
- net +12V: track 254.0 -> 114.4 mm, vias 5 -> 1
- net Net-(F3-Pad1): track 139.6 -> 0.00 mm, vias 2 -> 0
- net Net-(C1-Pad1): track 119.1 -> 0.00 mm, vias 2 -> 0
- net Net-(C9-Pad1): track 109.2 -> 0.00 mm
- net Net-(D13-Pad1): track 96.1 -> 0.00 mm, vias 1 -> 0
- net MCU_button_on_board: track 93.0 -> 0.00 mm
- net MCU_Uref_2.5v: track 102.3 -> 12.6 mm
- net MCU_system_status_LED: track 86.0 -> 0.00 mm
- net Net-(D16-Pad1): track 84.4 -> 0.00 mm, vias 3 -> 0
- net Net-(R46-Pad1): track 79.7 -> 0.00 mm
- net MCU_main_supply_enable: track 4.38 -> 76.5 mm, vias 0 -> 1
- net Net-(D15-Pad1): track 71.5 -> 0.00 mm, vias 2 -> 0
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- added copper zone on F.Cu, net 7.2V_stab

Commit message: update pcb
Parts:
- added L4: FB, Inductor_SMD:L_1206_3216Metric_Pad1.42x1.75mm_HandSolder, B.Cu at (153.4, 75.1)
- D22, D23, D25, D26, D27, R22: moved to F.Cu
- L2, L3: moved to B.Cu
- moved D13 87.6 mm to (114.5, 94.0), turned to 270 degrees
- moved R11 85.4 mm to (116.9, 93.1), turned to 270 degrees
- moved R15 82.8 mm to (119.1, 93.1), turned to 270 degrees
- moved D19 79.3 mm to (121.4, 93.9), turned to 270 degrees
- moved R33 77.0 mm to (136.0, 112.6)
- moved D21 65.0 mm to (151.8, 84.1), turned to 180 degrees
- moved L2 64.6 mm to (142.1, 60.3), turned to 180 degrees
- moved R12 63.5 mm to (133.6, 94.5), turned to 270 degrees
- moved R50 62.2 mm to (118.7, 115.3)
- moved D14 62.0 mm to (130.9, 96.1), turned to 270 degrees
- moved Q2 61.7 mm to (122.0, 115.3)
- moved R49 60.9 mm to (116.4, 115.3), turned to 270 degrees
- moved R16 60.6 mm to (135.7, 94.5), turned to 270 degrees
- moved D16 60.4 mm to (146.4, 100.5)
- moved R51 58.6 mm to (125.5, 115.2)
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Connections:
- C29 pad 1: +5v_FROM_MCU -> Net-(C29-Pad1)
- R58 pad 2: +5v_FROM_MCU -> Net-(C29-Pad1)
Routing:
- net +5v_FROM_MCU: track 55.3 -> 213.6 mm, vias 2 -> 12
- net Net-(C30-Pad1): track 0.00 -> 98.6 mm, vias 0 -> 5
- net LOW_WASHER_WATER_LEVEL_INPUT: track 0.00 -> 98.1 mm, vias 0 -> 2
- net WATER_FLOW_SENSOR_INPUT: track 0.00 -> 94.8 mm, vias 0 -> 2
- net GND: track 404.0 -> 490.2 mm, vias 5 -> 20
- net IGNITION_SWITCH_INPUT: track 0.00 -> 79.4 mm, vias 0 -> 2
- net PROXIMITY_SENSOR_INPUT: track 0.00 -> 59.7 mm, vias 0 -> 2
- net SPARE_INPUT_1: track 0.00 -> 56.1 mm, vias 0 -> 2
- net DOOR_SWITCH_INPUT: track 0.00 -> 53.4 mm, vias 0 -> 2
- net MCU_button_on_board: track 0.00 -> 37.5 mm, vias 0 -> 4
- net MCU_pjon_bus_PIN: track 9.89 -> 46.0 mm, vias 0 -> 1
- net MCU_sensors_voltage_test_input: track 0.00 -> 28.7 mm, vias 0 -> 2
- net MCU_UART1_TX: track 0.00 -> 25.3 mm, vias 0 -> 2
- net MCU_UART1_RX: track 0.00 -> 22.5 mm
- net Net-(C35-Pad1): track 0.00 -> 19.4 mm
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Other:
- copper layers 2 -> 4
- net class gnd: clearance 0.2 -> 0.3

Commit message: pcb
Parts:
- moved R65 11.2 mm to (131.8, 92.6), turned to 270 degrees
- moved R22 7.50 mm to (151.0, 105.6)
- moved D37 0.31 mm to (116.0, 122.0)
- turned R44 to 0 degrees
Routing:
- net Net-(C23-Pad1): track 5.60 -> 223.6 mm, vias 0 -> 4
- net GND: track 490.2 -> 643.4 mm, vias 20 -> 39
- net +5v_FROM_MCU: track 213.6 -> 362.4 mm, vias 12 -> 20
- net MCU_system_status_LED: track 0.00 -> 100.4 mm, vias 0 -> 4
- net +12V: track 119.4 -> 215.3 mm, vias 1 -> 5
- net MCU_UART2_RX: track 0.00 -> 91.8 mm, vias 0 -> 7
- net Net-(F3-Pad1): track 0.00 -> 86.3 mm, vias 0 -> 4
- net Net-(R46-Pad1): track 0.00 -> 84.2 mm, vias 0 -> 3
- net MCU_spare_input_1: track 0.00 -> 83.0 mm, vias 0 -> 6
- net Net-(R47-Pad1): track 0.00 -> 78.8 mm, vias 0 -> 3
- net MCU_spare_out_1: track 0.00 -> 69.6 mm, vias 0 -> 4
- net MCU_UART2_TX: track 0.00 -> 67.5 mm, vias 0 -> 6
- net MCU_converter_out: track 0.00 -> 67.0 mm, vias 0 -> 4
- net MCU_light_out: track 0.00 -> 65.7 mm, vias 0 -> 3
- net Net-(R48-Pad1): track 0.00 -> 65.2 mm
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- added copper zone on In2.Cu, net GND
Other:
- board text added: "+5S"
- board text added: "+B"
- board text added: "1Wire"
- board text added: "A"
- board text added: "B"
- board text added: "CONVERTER"
- board text added: "DOOR"
- board text added: "EN"
- board text added: "Encoder"
- board text added: "Flow S"
- board text added: "GND"
- board text added: "I2C"
- board text added: "IGN"
- board text added: "LCD SPI"
- board text added: "LIGHT"
- board text added: "Low Wash"
- board text added: "Outputs"
- board text added: "PJON"
- board text added: "PRX S"
- board text added: "PUMP"
- board text added: "RS485"
- board text added: "Resist Sens"
- board text added: "Spare"
- board text added: "Uart 1"

Commit message: Pcb and shematic changed
Other:
- board text added: "CAR BS CONTROLLER V3"

Commit message: update
Parts:
- R1: value 2k2 -> 3k9
- R22: value 3k -> 2k2
- R27: value 1k -> (not used) 1k
- R32: value 1k2 -> 2k2
- R56: value 1k -> 2k*
- R62: value 10k -> 10k*
- R64: value 10k -> 15k*
- U6: value MCP6004 -> MCP6004(LM324)
