File: KiCad/Cbc_power_supply_module/Cbc_power_supply_module.sch (KiCad schematic (older format))
At the start: 30 parts, among them J1 Conn_01x05, J2 Conn_01x04, U1 NCP3064B, U2 NCP3064B

Commit message: update
Parts:
- renumbered R8 to R8*
Changed lines of the file:
@@
 	6150 1850 6150 1800
 $Comp
-L Device:R R8
+L Device:R R8*
 U 1 1 6081683A
 P 6150 2000
-F 0 "R8" H 6080 1954 50  0000 R CNN
+F 0 "R8*" H 6080 1954 50  0000 R CNN
 F 1 "12k" H 6080 2045 50  0000 R CNN
 F 2 "Resistor_SMD:R_0805_2012Metric_Pad1.20x1.40mm_HandSolder" V 6080 2000 50  0001 C CNN
